File: 18f-blinkie.kicad_pcb (KiCad board)
At the start: 2 copper layers, 96.5 x 94 mm, 21 parts, among them J1 Conn_01x07_Female, J2 Conn_01x07_Female

Commit message: Removed resistors, submitted.
Parts:
- removed R1, R2, R3, R4, R5, R6: 220R, Resistor_SMD:R_0805_2012Metric_Pad1.20x1.40mm_HandSolder
- added REF**: OSHW-Logo2_14.6x12mm_SilkScreen, Symbol:OSHW-Logo2_14.6x12mm_SilkScreen, B.Cu at (177.8, 137.4)
Connections:
- D1 pad 1: Net-(D1-Pad1) -> 5V
- D2 pad 1: Net-(D2-Pad1) -> 5V
- D3 pad 1: Net-(D3-Pad1) -> 5V
- D4 pad 1: Net-(D4-Pad1) -> 5V
- D5 pad 1: Net-(D5-Pad1) -> 5V
- D6 pad 1: Net-(D6-Pad1) -> 5V
Routing:
- net 5V: track 431.4 -> 450.8 mm, vias 2 -> 10
- net GND: track 472.8 -> 455.7 mm
- net Net-(D2-Pad1): track 15.2 -> 0.00 mm, vias 1 -> 0
- net Net-(D6-Pad1): track 13.8 -> 0.00 mm, vias 1 -> 0
- net Net-(D1-Pad1): track 11.7 -> 0.00 mm, vias 1 -> 0
- net Net-(D4-Pad1): track 11.5 -> 0.00 mm, vias 1 -> 0
- net Net-(D5-Pad1): track 10.7 -> 0.00 mm, vias 1 -> 0
- net Net-(D3-Pad1): track 7.53 -> 0.00 mm, vias 1 -> 0
- net DATA: track 44.2 -> 42.2 mm
- net Net-(D2-Pad2): track 107.5 -> 108.2 mm
- net Net-(D1-Pad2): track 95.3 -> 94.7 mm
- added copper zone on B.Cu, net (none)
- added copper zone on F.Cu, net (none)
